Commit message: added gps, imu and oak to urdf

File: urdf/roboclaw_description.urdf.xacro (robot description, xacro)
@@ -14,4 +14,8 @@
   <xacro:property name="caster_wheel_mass" value="0.1" /> <!-- TODO: Fixme -->
   <xacro:property name="caster_wheel_radius" value="0.128" />
+  <xacro:property name="oak_z" value ="0.5"/>
+  <xacro:property name="oak_x" value ="0.15"/>
+  <xacro:property name="oak_r" value ="0.0"/>
+  <xacro:property name="oak_p" value ="0.54"/>
   <link name="base_footprint" />
   <joint name="base_joint" type="fixed">
@@ -101,6 +105,6 @@
           iyy="${wheel_mass / 12.0 * wheel_radius*wheel_radius}" iyz="0.0"
           izz="${wheel_mass / 12.0 * wheel_radius*wheel_radius}"/>
-        </inertial>
-      </link>
+      </inertial>
+    </link>
     <joint name="caster_left_wheel_joint" type="fixed">
       <parent link="base_link"/>
@@ -158,5 +162,67 @@
           izz="${caster_wheel_mass * 0.4 * (caster_wheel_radius * caster_wheel_radius)}"/>
         </inertial>
-      </link>
+    </link>
+      <!-- start -->
+       <!-- *********************** IMU SETUP *********************************  -->
+  <!-- Each sensor must be attached to a link.                              -->
+  <!-- *********************** GPS SETUP **********************************  -->
+    <joint name="gps_joint" type="fixed">
+      <parent link="base_link"/>
+      <child link="gps_link"/>
+      <origin xyz="0.0 0 0.8" rpy="0 0 0"/>
+    </joint>
+    <link name="gps_link">
+      <visual name="">
+              <origin xyz="0.0 0.0 0.0" rpy="0.0 0.0 0.0"/>
+              <geometry>
+                  <cylinder radius="0.1" length="0.1"/>
+              </geometry>
+              <material name="purple">
+                  <color rgba="1.0 0.0 1.0 1.0"/>
+                  <texture filename=""/>
+              </material>
+        </visual>
+    </link>
+    <!-- *********************** OAK SETUP **********************************  -->
+    <joint name="oak_joint" type="fixed">
+      <parent link="base_link"/>
+      <child link="oak_link"/>
+      <origin xyz="${oak_x} 0 ${oak_z}" rpy="${oak_r} ${oak_p} 0"/>
+    </joint>
+    <link name="oak_link">
+      <visual name="">
+          <origin xyz="0. 0.0 0.0" rpy="0.0 0.0 0.0"/>
+          <geometry>
+              <!-- <cylinder radius="0.1" length="0.1"/> -->
+              <box size=".1 .4 .1"/>
+          </geometry>
+          <material name="notsure">
+              <color rgba="0.5 0.5 0.5 1.0"/>
+              <texture filename=""/>
+          </material>
+      </visual>
+    </link>
+        <!-- oak optical -->
+    <joint name="oak_opt_joint" type="fixed">
+        <parent link="oak_link"/>
+        <!-- <child link="oak_opt_link"/> -->
+        <child link="oak-d-base-frame"/>
+        <origin xyz=".1 0 0 " rpy="${0*pi/2} ${-pi/10} ${0*pi/2}"/>
+    </joint>
+      <!-- <link name="oak_opt_link"> -->
+    <link name="oak-d-base-frame">
+        <visual name="">
+            <origin xyz="0. 0.0 0.0" rpy="0.0 0.0 0.0"/>
+            <geometry>
+                <cylinder radius="0.1" length="0.1"/>
+                <!-- <box size=".1 .4 .1"/> -->
+            </geometry>
+            <material name="notsure">
+                <color rgba="1.0 0.5 0.5 1.0"/>
+                <texture filename=""/>
+            </material>
+        </visual>
+    </link>
+      <!-- end -->
   </xacro:macro>
 </robot>

Commit message: added camera and imu

File: urdf/roboclaw_description.urdf.xacro (robot description, xacro)
@@ -165,5 +165,22 @@
       <!-- start -->
        <!-- *********************** IMU SETUP *********************************  -->
-  <!-- Each sensor must be attached to a link.                              -->
+  <!--Each sensor must be attached to a link.        -->
+    <joint name="imu_joint" type="fixed">
+      <parent link="base_link"/>
+      <child link="imu_link"/>
+      <origin xyz="-0.00 0 0.2" rpy="0 0 0"/>
+    </joint>
+    <link name="imu_link">
+  <visual name="">
+              <origin xyz="0.0 0.0 0.0" rpy="0.0 0.0 0.0"/>
+              <geometry>
+                  <cylinder radius="0.1" length="0.1"/>
+              </geometry>
+              <material name="not_purple">
+                  <color rgba="0.0 0.0 1.0 1.0"/>
+                  <texture filename=""/>
+              </material>
+          </visual>
+      </link>
   <!-- *********************** GPS SETUP **********************************  -->
     <joint name="gps_joint" type="fixed">
@@ -179,4 +196,22 @@
               </geometry>
               <material name="purple">
+                  <color rgba="1.0 0.0 1.0 1.0"/>
+                  <texture filename=""/>
+              </material>
+        </visual>
+    </link>
+    <!-- *********************** Camera SETUP **********************************  -->
+    <joint name="camera_joint" type="fixed">
+      <parent link="base_link"/>
+      <child link="camera_link"/>
+      <origin xyz="0.4 0 0.8" rpy="0 0 0.18"/>
+    </joint>
+    <link name="camera_link">
+      <visual name="">
+              <origin xyz="0.0 0.0 0.0" rpy="0.0 0.0 0.0"/>
+              <geometry>
+                  <cylinder radius="0.1" length="0.1"/>
+              </geometry>
+              <material name="white">
                   <color rgba="1.0 0.0 1.0 1.0"/>
                   <texture filename=""/>

Commit message: fixed camera orientation

File: urdf/roboclaw_description.urdf.xacro (robot description, xacro)
@@ -205,5 +205,5 @@
       <parent link="base_link"/>
       <child link="camera_link"/>
-      <origin xyz="0.4 0 0.8" rpy="0 0 0.18"/>
+      <origin xyz="0.4 0 0.8" rpy="0 0.18 0"/>
     </joint>
     <link name="camera_link">
